Commit message: changes the value

File: src/my_robot_description/urdf/my_base.urdf (robot description, URDF)
Before this commit: robot sophus, 2 links, 1 joints
Links:
- removed link wheel_link
- added link stepper_motor, mass 0.15; collision mesh filename=package://my_robot_description/meshes/nema17_17HS4401_b.stl scale=9 9 9; visual mesh filename=package://my_robot_description/meshes/nema17_17HS4401_b.stl scale=9 9 9
- added link wheel, mass 0.1; collision mesh filename=package://my_robot_description/meshes/wheel_v1.stl scale=0.01 0.01 0.01; visual mesh filename=package://my_robot_description/meshes/wheel_v1.stl scale=0.01 0.01 0.01
Joints:
- removed joint wheel_joint
- added joint motor_joint_right: type fixed, parent base_link, child stepper_motor, origin xyz=0.85 -0.22 0.26 rpy=0 1.57 0, axis 0 0 0
- added joint wheel_joint_right: type continuous, parent stepper_motor, child wheel, origin xyz=0 0 0.26 rpy=0 -3.14 0, axis 0 0 1

Commit message: change the axis of robot to standard format

File: src/my_robot_description/urdf/my_base.urdf (robot description, URDF)
Before this commit: robot sophus, 3 links, 2 joints
Joints:
- joint motor_joint_right: origin xyz=0.85 -0.22 0.26 rpy=0 1.57 0 -> xyz=-0.22 -0.85 0.295 rpy=1.57 0 0
- joint wheel_joint_right: origin xyz=0 0 0.26 rpy=0 -3.14 0 -> xyz=0 0 0.026 rpy=0 -3.14 0
