Commit message: add extra link and upgrade

File: src/my_robot_description/urdf/my_robot.urdf (robot description, URDF)
Before this commit: robot cylinder_stack, 3 links, 2 joints
Links:
- added link link0, mass 1.0; collision cylinder length=0.5 radius=0.1; visual cylinder length=0.1 radius=0.1
- link base_link: mass 1.0 -> 0.5; geometry collision cylinder length=0.5 radius=0.2; visual cylinder length=0.05 radius=0.2
- link link1: geometry collision cylinder length=0.4 radius=0.05; visual cylinder length=0.4 radius=0.05
- link link2: geometry collision cylinder length=0.2 radius=0.04; visual cylinder length=0.4 radius=0.04
Joints:
- added joint joint0: type continuous, parent base_link, child link0, origin xyz=0 0 0.05 rpy=0 0 0, axis 0 0 1
- joint joint1: limit lower=-1.57 upper=1.57 effort=10 velocity=1 -> lower=0 upper=1.57 effort=10 velocity=1; origin xyz=0 0 0.025 rpy=0 0 0 -> xyz=0 0 0.1 rpy=0 0 0; parent base_link -> link0
- joint joint2: axis 0 0 1 -> 0 1 0; limit lower=-1.57 upper=1.57 effort=10 velocity=1 -> lower=0 upper=1.57 effort=10 velocity=1; origin xyz=0 0 0.3 rpy=0 0 0 -> xyz=0 0 0.4 rpy=0 0 0
