Commit message: update axis of robot to standard format of ros x-axis to front

File: src/my_robot_description/urdf/sophus.urdf.xacro (robot description, xacro)
@@ -1,7 +1,7 @@
 <?xml version="1.0"?>
 <robot name="sophus" xmlns:xacro="http://www.ros.org/wiki/xacro">
-    <xacro:property name="wheel_x" value="0.85"/>
-    <xacro:property name="wheel_y" value="-0.22"/>
-    <xacro:property name="wheel_z" value="-0.26"/>
+    <xacro:property name="wheel_x" value="-0.22"/>
+    <xacro:property name="wheel_y" value="-0.85"/>
+    <xacro:property name="wheel_z" value="0.295"/>
     <xacro:property name="wheel_caster" value="-0.26"/>
     <xacro:property name="motor_rotation" value="1.57"/>
@@ -12,10 +12,10 @@
                 <mesh filename="package://my_robot_description/meshes/base_plate_v1.stl" scale="0.01 0.01 0.01"/>
             </geometry>
-            <origin xyz="0 0 0" rpy="0 3.14 0"/>
+            <origin xyz="0 0 0.57" rpy="3.142 0 1.5708"/>
             <material name="black"><color rgba="0.1 0.1 0.1 1"/></material>
         </visual>
         <collision>
             <geometry>
-                <mesh filename="package://my_robot_description/meshes/base_plate_v1.stl" scale="0.01 0.01 0.01"/>
+                <mesh filename="package://my_robot_description/meshes/base_plate_v1.stl" scale="0.001 0.001 0.001"/>
             </geometry>
         </collision>
@@ -50,5 +50,5 @@
                 </geometry>
                 <origin xyz="0 0 0" rpy="0 0 0"/>
-                <material name="black"><color rgba="0.1 0.1 0.1 1"/></material>
+                <material name="red"><color rgba="0.9 0 0 1"/></material>
             </visual>
             <collision>
@@ -65,5 +65,5 @@
             <parent link="base_link"/>
             <child link="stepper_motor_${side}"/>
-            <origin xyz="${reflect*wheel_x} ${wheel_y} ${wheel_z}" rpy="0 ${reflect*motor_rotation} 0"/>
+            <origin xyz="${wheel_x} ${reflect*wheel_y} ${wheel_z}" rpy="${reflect*motor_rotation} 0 0"/>
             <axis xyz="0 0 0"/>
         </joint>
@@ -71,5 +71,5 @@
             <parent link="stepper_motor_${side}"/>
             <child link="wheel_${side}"/>
-            <origin xyz="0 0 0.26" rpy="0 ${reflect*wheel_rotation} 0"/>
+            <origin xyz="0 0 0.22" rpy="0 ${reflect*wheel_rotation} 0"/>
             <axis xyz="0 0 1"/>
         </joint>
@@ -78,12 +78,12 @@
         <visual>
             <geometry>
-                <mesh filename="package://my_robot_description/meshes/Caster_Wheel_V2.stl" scale="8.5 8.5 8.5"/>
+                <mesh filename="package://my_robot_description/meshes/Caster_Wheel_V2.stl" scale="7.5 7.5 7.5"/>
             </geometry>
             <origin xyz="0 0 0" rpy="0 0 0"/>
-            <material name="black"><color rgba="0.1 0.1 0.1 1"/></material>
+            <material name="green"><color rgba="0 0.9 0 1"/></material>
         </visual>
         <collision>
             <geometry>
-                <mesh filename="package://my_robot_description/meshes/Caster_Wheel_V2.stl" scale="8.5 8.5 8.5"/>
+                <mesh filename="package://my_robot_description/meshes/Caster_Wheel_V2.stl" scale="7.5 7.5 7.5"/>
             </geometry>
         </collision>
@@ -96,5 +96,5 @@
         <parent link="base_link"/>
         <child link="caster_wheel"/>
-        <origin xyz="0 1.02 -0.22" rpy="0 0 0"/>
+        <origin xyz="1.03 0 0.36" rpy="0 0 1.57"/>
         <axis xyz="0 0 1"/>
     </joint>

File: src/my_robot_description/urdf/sophus_core.xacro (robot description, xacro)
@@ -1,7 +1,7 @@
 <?xml version="1.0"?>
 <robot xmlns:xacro="http://www.ros.org/wiki/xacro">
-    <xacro:property name="wheel_x" value="0.085"/>
-    <xacro:property name="wheel_y" value="-0.022"/>
-    <xacro:property name="wheel_z" value="-0.026"/>
+    <xacro:property name="wheel_x" value="-0.22"/>
+    <xacro:property name="wheel_y" value="-0.85"/>
+    <xacro:property name="wheel_z" value="0.295"/>
     <xacro:property name="wheel_caster" value="-0.26"/>
     <xacro:property name="motor_rotation" value="1.57"/>
@@ -10,12 +10,13 @@
         <visual>
             <geometry>
-                <mesh filename="package://my_robot_description/meshes/base_plate_v1.stl" scale="0.001 0.001 0.001"/>
+                <mesh filename="package://my_robot_description/meshes/base_plate_v1.stl" scale="0.01 0.01 0.01"/>
             </geometry>
-            <origin xyz="0 0 0" rpy="0 3.14 0"/>
+            <origin xyz="0 0 0.57" rpy="3.142 0 1.5708"/>
             <material name="black"><color rgba="0.1 0.1 0.1 1"/></material>
         </visual>
         <collision>
+            <origin xyz="0 0 0.57" rpy="3.142 0 1.5708"/>
             <geometry>
-                <mesh filename="package://my_robot_description/meshes/base_plate_v1.stl" scale="0.001 0.001 0.001"/>
+                <mesh filename="package://my_robot_description/meshes/base_plate_v1.stl" scale="0.01 0.01 0.01"/>
             </geometry>
         </collision>
@@ -29,5 +30,5 @@
             <visual>
                 <geometry>
-                    <mesh filename="package://my_robot_description/meshes/nema17_17HS4401_b.stl" scale="1 1 1"/>
+                    <mesh filename="package://my_robot_description/meshes/nema17_17HS4401_b.stl" scale="9 9 9"/>
                 </geometry>
                 <origin xyz="0 0 0" rpy="0 0 0"/>
@@ -36,5 +37,5 @@
             <collision>
                 <geometry>
-                    <mesh filename="package://my_robot_description/meshes/nema17_17HS4401_b.stl" scale="1 1 1"/>
+                    <mesh filename="package://my_robot_description/meshes/nema17_17HS4401_b.stl" scale="9 9 9"/>
                 </geometry>
             </collision>
@@ -47,5 +48,5 @@
             <visual>
                 <geometry>
-                    <mesh filename="package://my_robot_description/meshes/wheel_v1.stl" scale="0.001 0.001 0.001"/>
+                    <mesh filename="package://my_robot_description/meshes/wheel_v1.stl" scale="0.01 0.01 0.01"/>
                 </geometry>
                 <origin xyz="0 0 0" rpy="0 0 0"/>
@@ -54,5 +55,5 @@
             <collision>
                 <geometry>
-                    <mesh filename="package://my_robot_description/meshes/wheel_v1.stl" scale="0.001 0.001 0.001"/>
+                    <mesh filename="package://my_robot_description/meshes/wheel_v1.stl" scale="0.01 0.01 0.01"/>
                 </geometry>
             </collision>
@@ -65,14 +66,12 @@
             <parent link="base_link"/>
             <child link="stepper_motor_${side}"/>
-            <origin xyz="${reflect*wheel_x} ${wheel_y} ${wheel_z}" rpy="0 ${reflect*motor_rotation} 0"/>
+            <origin xyz="${reflect*wheel_x} ${wheel_y} ${wheel_z}" rpy="${reflect*motor_rotation} 0 0"/>
             <axis xyz="0 0 0"/>
         </joint>
-        <joint name="wheel_joint_${side}" type="revolute">
+        <joint name="wheel_joint_${side}" type="continuous">
             <parent link="stepper_motor_${side}"/>
             <child link="wheel_${side}"/>
             <origin xyz="0 0 0.026" rpy="0 ${reflect*wheel_rotation} 0"/>
             <axis xyz="0 0 1"/>
-            <limit effort="20" velocity="30"/>
-            <dynamics damping="0.1" friction="0.0"/>
         </joint>
     </xacro:macro>

Commit message: update the property and inertia

File: src/my_robot_description/urdf/sophus.urdf.xacro (robot description, xacro)
@@ -1,10 +1,29 @@
 <?xml version="1.0"?>
 <robot name="sophus" xmlns:xacro="http://www.ros.org/wiki/xacro">
+    <!-- ===================== Geometry properties ===================== -->
     <xacro:property name="wheel_x" value="-0.22"/>
     <xacro:property name="wheel_y" value="-0.85"/>
     <xacro:property name="wheel_z" value="0.295"/>
-    <xacro:property name="wheel_caster" value="-0.26"/>
-    <xacro:property name="motor_rotation" value="1.57"/>
-    <xacro:property name="wheel_rotation" value="-3.14"/>
+    <xacro:property name="wheel_offset" value="0.22"/>            <!-- shaft offset motor -> wheel -->
+    <xacro:property name="wheel_half_track" value="${0.85 + wheel_offset}"/>  <!-- = 1.07 m, centre -> wheel -->
+    <xacro:property name="wheel_radius" value="0.295"/>           <!-- = wheel centre height, so wheel touches ground -->
+    <xacro:property name="wheel_width"  value="0.15"/>            <!-- thickness of wheel along its axis -->
+    <xacro:property name="caster_radius" value="0.10"/>
+    <xacro:property name="caster_z_offset" value="-0.26"/>        <!-- caster ball centre = 0.36-0.26 = 0.10 above ground -->
+    <!-- Base mesh pose (same pose is used for visual AND collision) -->
+    <xacro:property name="base_mesh_xyz" value="0 0 0.57"/>
+    <xacro:property name="base_mesh_rpy" value="3.142 0 1.5708"/>
+    <!-- ===================== Inertia helper ===================== -->
+    <xacro:macro name="cylinder_inertial" params="m r h">
+        <inertial>
+            <mass value="${m}"/>
+            <inertia ixx="${m*(3*r*r+h*h)/12}" ixy="0" ixz="0"
+                     iyy="${m*(3*r*r+h*h)/12}" iyz="0"
+                     izz="${m*r*r/2}"/>
+        </inertial>
+    </xacro:macro>
+    <!-- ===================== Base ===================== -->
+    <!-- base_link is the root (dummy_link removed: it would give base_link two TF parents
+         once Gazebo publishes odom -> base_link) -->
     <link name="base_link">
         <visual>
@@ -12,18 +31,24 @@
                 <mesh filename="package://my_robot_description/meshes/base_plate_v1.stl" scale="0.01 0.01 0.01"/>
             </geometry>
-            <origin xyz="0 0 0.57" rpy="3.142 0 1.5708"/>
+            <origin xyz="${base_mesh_xyz}" rpy="${base_mesh_rpy}"/>
             <material name="black"><color rgba="0.1 0.1 0.1 1"/></material>
         </visual>
         <collision>
             <geometry>
-                <mesh filename="package://my_robot_description/meshes/base_plate_v1.stl" scale="0.001 0.001 0.001"/>
+                <mesh filename="package://my_robot_description/meshes/base_plate_v1.stl" scale="0.01 0.01 0.01"/>
             </geometry>
+            <!-- FIX: collision now has the SAME origin as the visual (it was missing before) -->
+            <origin xyz="${base_mesh_xyz}" rpy="${base_mesh_rpy}"/>
         </collision>
+        <!-- Realistic mass/inertia (approx. 1.2 x 1.0 x 0.3 m box, 10 kg) -->
         <inertial>
-            <mass value="0.15"/>
-            <inertia ixx="0.0001" ixy="0" ixz="0" iyy="0.0001" iyz="0" izz="0.0001"/>
+            <origin xyz="0 0 0.35" rpy="0 0 0"/>
+            <mass value="10.0"/>
+            <inertia ixx="0.91" ixy="0" ixz="0" iyy="1.28" iyz="0" izz="2.03"/>
         </inertial>
     </link>
+    <!-- ===================== Wheel assembly ===================== -->
     <xacro:macro name="wheel_assembly" params="side reflect">
+        <!-- Motor: visual only (no collision needed) -->
         <link name="stepper_motor_${side}">
             <visual>
@@ -34,12 +59,7 @@
                 <material name="grey"><color rgba="0.4 0.4 0.4 1"/></material>
             </visual>
-            <collision>
-                <geometry>
-                    <mesh filename="package://my_robot_description/meshes/nema17_17HS4401_b.stl" scale="9 9 9"/>
-                </geometry>
-            </collision>
             <inertial>
-                <mass value="0.15"/>
-                <inertia ixx="0.0001" ixy="0" ixz="0" iyy="0.0001" iyz="0" izz="0.0001"/>
+                <mass value="0.5"/>
+                <inertia ixx="0.005" ixy="0" ixz="0" iyy="0.005" iyz="0" izz="0.005"/>
             </inertial>
         </link>
@@ -52,27 +72,28 @@
                 <material name="red"><color rgba="0.9 0 0 1"/></material>
             </visual>
+            <!-- FIX: simple cylinder collision (axis = link z = joint axis) instead of the STL -->
             <collision>
                 <geometry>
-                    <mesh filename="package://my_robot_description/meshes/wheel_v1.stl" scale="0.01 0.01 0.01"/>
+                    <cylinder radius="${wheel_radius}" length="${wheel_width}"/>
                 </geometry>
             </collision>
-            <inertial>
-                <mass value="0.1"/>
-                <inertia ixx="0.0001" ixy="0" ixz="0" iyy="0.0001" iyz="0" izz="0.0001"/>
-            </inertial>
+            <xacro:cylinder_inertial m="1.0" r="${wheel_radius}" h="${wheel_width}"/>
         </link>
         <joint name="motor_joint_${side}" type="fixed">
             <parent link="base_link"/>
             <child link="stepper_motor_${side}"/>
-            <origin xyz="${wheel_x} ${reflect*wheel_y} ${wheel_z}" rpy="${reflect*motor_rotation} 0 0"/>
-            <axis xyz="0 0 0"/>
+            <origin xyz="${wheel_x} ${reflect*wheel_y} ${wheel_z}" rpy="${reflect*pi/2} 0 0"/>
         </joint>
         <joint name="wheel_joint_${side}" type="continuous">
             <parent link="stepper_motor_${side}"/>
             <child link="wheel_${side}"/>
-            <origin xyz="0 0 0.22" rpy="0 ${reflect*wheel_rotation} 0"/>
-            <axis xyz="0 0 1"/>
+            <origin xyz="0 0 ${wheel_offset}" rpy="0 ${reflect*pi} 0"/>
+            <!-- FIX: axis now points along +Y of base_link for BOTH wheels
+                 (before: left = -Y, right = +Y -> wheels spun against each other) -->
+            <axis xyz="0 0 ${reflect}"/>
+            <dynamics damping="0.01" friction="0.0"/>
         </joint>
     </xacro:macro>
+    <!-- ===================== Caster ===================== -->
     <link name="caster_wheel">
         <visual>
@@ -83,12 +104,14 @@
             <material name="green"><color rgba="0 0.9 0 1"/></material>
         </visual>
+        <!-- FIX: frictionless sphere (friction set in the gazebo file) instead of STL mesh -->
         <collision>
             <geometry>
-                <mesh filename="package://my_robot_description/meshes/Caster_Wheel_V2.stl" scale="7.5 7.5 7.5"/>
+                <sphere radius="${caster_radius}"/>
             </geometry>
+            <origin xyz="0 0 ${caster_z_offset}" rpy="0 0 0"/>
         </collision>
         <inertial>
-            <mass value="0.15"/>
-            <inertia ixx="0.0001" ixy="0" ixz="0" iyy="0.0001" iyz="0" izz="0.0001"/>
+            <mass value="0.5"/>
+            <inertia ixx="0.002" ixy="0" ixz="0" iyy="0.002" iyz="0" izz="0.002"/>
         </inertial>
     </link>
@@ -97,5 +120,4 @@
         <child link="caster_wheel"/>
         <origin xyz="1.03 0 0.36" rpy="0 0 1.57"/>
-        <axis xyz="0 0 1"/>
     </joint>
     <xacro:wheel_assembly side="left"  reflect="-1"/>
